File: CircuitFiles/Lab5/Lab5.brd (EAGLE design)
At the start: 100 x 75 mm, 26 parts, among them IC1 LM4041CILPRCLP, U1 TLV5616, U2 MC34119

Commit message: Updating Labs 5 and 6
Parts:
- C3: value 0.1 -> 0.1 uF
Changed lines of the file:
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@@
 <element name="C1" library="EE445L" package="CAP200MILPOLARIZED" value="10 Uf" x="-2.54" y="-176.53"/>
 <element name="C2" library="EE445L" package="CAP200MIL" value="0.1 uF" x="-3.175" y="-182.88"/>
-<element name="C3" library="EE445L" package="CAP200MIL" value="0.1" x="-3.175" y="-187.325"/>
+<element name="C3" library="EE445L" package="CAP200MIL" value="0.1 uF" x="-3.175" y="-187.325"/>
 <element name="C4" library="EE445L" package="CAP200MILPOLARIZED" value="4.7 uF" x="-2.54" y="-192.405"/>
 <element name="R6" library="EE445L" package="RES300MIL" value="20K" x="-1.905" y="-198.755"/>
