File: CircuitFiles/Lab5/Lab5.sch (EAGLE design)
At the start: 26 parts, among them IC1 LM4041CILPRCLP, U1 TLV5616, U2 MC34119

Commit message: Updating Labs 5 and 6
Parts:
- C3: value 0.1 -> 0.1 uF
Changed lines of the file:
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@@
 <part name="C1" library="EE445L" deviceset="CAPACITOR_POLARIZED" device="E5-6" value="10 Uf"/>
 <part name="C2" library="EE445L" deviceset="CAPACITOR" device="050-024X044" value="0.1 uF"/>
-<part name="C3" library="EE445L" deviceset="CAPACITOR" device="050-024X044" value="0.1"/>
+<part name="C3" library="EE445L" deviceset="CAPACITOR" device="050-024X044" value="0.1 uF"/>
 <part name="C4" library="EE445L" deviceset="CAPACITOR_POLARIZED" device="E5-6" value="4.7 uF"/>
 <part name="SUPPLY3" library="EE445L" deviceset="GND" device=""/>
