File: CircuitFiles/Lab7/Lab7.sch (EAGLE design)
At the start: 28 parts, among them IC1 LM7805, Q1 PN2222, Q2 PN2222, Q3 IRF522, Q4 IRF522, Q5 FQP27P06, Q6 FQP27P06

Commit message: Updating lab 7 stuff and adding lab 8 report
Parts:
- removed +3.3V, +5V, GND: TP2, EE445L:TP2
- removed Q3, Q4: IRF522, transistor-power:IRF3704-H
- removed Q5, Q6: FQP27P06, transistor-power:IRF4905
- removed TILT_BACK, TILT_FOR: (no value), EE445L:B3F-1052
- added BATTERY: (no value), EE445L:PINHD-1X2/90
- added DECREASE, INCREASE: (no value), EE445L:B3F-1052
- added ENC_MOTOR2: (no value), EE445L:PINHD-1X6
- added IC2, IC3, IC4, IC5, IC6, IC7, IC8, IC9: LM7805, EE445L:78XXS
- added Q7, Q8: PN2222, EE445L:PN2222
- added R11, R12, R13, R14: 10k, EE445L:RESISTOR0204/7
- added R6, R8: 1k, EE445L:RESISTOR0204/7
- added TILT_SWITCHES: (no value), switch-dil:DIP02YL
- R7: device rcl:R-US_0204/2V -> EE445L:RESISTOR0204/7
- U$1: value EK-TM4C1294XL_BOOST2 -> EK-TM4C1294XL_BOOST1; device EE445L:EK-TM4C1294XL_BOOST2 -> EE445L:EK-TM4C1294XL_BOOST1
- U$2: value EK-TM4C1294XL_BOOST1 -> EK-TM4C1294XL_BOOST2; device EE445L:EK-TM4C1294XL_BOOST1 -> EE445L:EK-TM4C1294XL_BOOST2
- renumbered NXT_MOTOR to ENC_MOTOR1
Connections:
- removed net +3.3V: +3.3V.TPA, +3.3V.TPB, DIS1.LIGHT, DIS1.VCC, U$1.+3.3V
- removed net +VBATT: C2.1, ENC_MOTOR1.1, IC1.IN, Q5.S, Q6.S, R4.2, R5.2
- removed net ENC_A: ENC_MOTOR1.5
- removed net ENC_B: ENC_MOTOR1.6
- removed net M+: ENC_MOTOR1.3, Q3.D, Q5.D
- removed net M-: ENC_MOTOR1.4, Q4.D, Q6.D
- removed net N$1: R3.1
- removed net N$10: TILT_BACK.S
- removed net N$5: R9.2, TILT_FOR.S1
- removed net N$6: R10.2, TILT_BACK.S1
- removed net PB2: R7.2, START/STOP.S
- removed net PB3: TILT_FOR.S
- new net DECREMENT: DECREASE.S, DECREASE.S1, R14.2, U$1.PE3
- new net ENC_1A: ENC_MOTOR1.3, U$1.PL1
- new net ENC_1B: ENC_MOTOR1.4, U$1.PL2
- new net ENC_2A: ENC_MOTOR2.3
- new net ENC_2B: ENC_MOTOR2.4
- new net FORWARD1: IC2.OUT, IC3.OUT, Q7.C, R11.1
- new net INCREMENT: INCREASE.S, INCREASE.S1, R13.2, U$1.PE2
- new net M1-: ENC_MOTOR1.6, IC8.GND, IC9.GND
- new net M2+: ENC_MOTOR2.5, IC2.GND, IC3.GND
- new net M2-: ENC_MOTOR2.6, IC4.GND, IC5.GND
- new net N$11: ENC_MOTOR1.5, IC6.GND, IC7.GND
- new net N$8: Q7.B, R8.2
- new net N$9: Q8.B, R6.1
- new net NO: U$2.PQ3
- new net NOPE: U$2.PQ2
- new net PL3: U$1.PL3
- new net PWM1: R6.2, U$1.PF1
- new net PWM2: R8.1, U$1.PF2
- new net PWM3: R2.2, U$1.PF3
- new net PWM4: R3.1, U$1.PG0
- new net PWM5: U$2.PG1
- new net PWM6: U$2.PK4
- new net PWM7: U$2.PK5
- new net REVERSE1: IC4.OUT, IC5.OUT, Q8.C, R12.1
- new net START/STOP: R7.2, START/STOP.S, START/STOP.S1, U$1.PD7
- new net TILT_BACK: R10.2, TILT_SWITCHES.3, U$1.PE1
- new net TILT_FOR: R9.2, TILT_SWITCHES.4, U$1.PE0
- net +3V3: now also DIS1.LIGHT, DIS1.VCC, IC7.IN, IC9.IN, R4.2, R5.2, U$1.+3.3V, U$2.+3.3V; no longer START/STOP.P, TILT_BACK.P, TILT_FOR.P
- net +5V: now also DECREASE.P, DECREASE.P1, ENC_MOTOR1.1, ENC_MOTOR2.1, INCREASE.P, INCREASE.P1, START/STOP.P, START/STOP.P1, TILT_SWITCHES.1, TILT_SWITCHES.2, U$2.+5V; no longer +5V.TPA, +5V.TPB
- net FORWARD: now also IC6.OUT, IC7.OUT; no longer Q3.G, Q5.G
- net GND: now also BATTERY.2, ENC_MOTOR2.2, IC3.IN, IC4.IN, IC6.IN, IC8.IN, Q7.E, Q8.E, R13.1, R14.1, U$1.GND2, U$2.GND, U$2.GND2; no longer GND.TPA, GND.TPB, Q3.S, Q4.S
- net N$2: now also BATTERY.1, C2.1, IC1.IN, IC2.IN, IC5.IN, R11.2, R12.2; no longer R2.2
- net PA2: now also U$1.PD0; no longer U$1.PQ3
- net PA3: now also U$1.PD1; no longer U$1.PQ2
- net PA4: now also U$1.PM4, U$2.PA4; no longer U$1.PA4
- net PA5: now also U$1.PM5, U$2.PA5; no longer U$1.PA5
- net PA6: now also U$1.PA6; no longer U$2.PA6
- net PA7: now also U$1.PH3, U$2.PA7; no longer U$1.PA7
- net REVERSE: now also IC8.OUT, IC9.OUT; no longer Q4.G, Q6.G
Other:
- moved on the sheet: U$2
